File: prototype/prototype.kicad_sch (KiCad schematic)
At the start: 0 parts

Commit message: feat: add kicad project
Other:
- company: (none) -> Ryoga.exe
- title: (none) -> UniSlider Prototype
Changed lines of the file:
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@@
 	(generator_version "9.0")
 	(paper "A4")
+	(title_block
+		(title "UniSlider Prototype")
+		(date "2025-10-05")
+		(company "Ryoga.exe")
+	)
 	(sheet_instances
 		(path "/"
